File: _autosave-555_Badge.kicad_pcb (KiCad board)
At the start: 2 copper layers, 53.8 x 85.6 mm, 15 parts, among them Q1 2N3904, U1 7555

Commit message: Everything looks amazing. PCB is basically done. Just need to generate a gerber file
Parts:
- moved R3 99.8 mm to (174.6, 110.5), turned to 90 degrees
- moved R5 96.0 mm to (171.4, 114.9)
- moved R6 89.7 mm to (167.0, 110.5), turned to 90 degrees
- moved S1 89.1 mm to (154.9, 108.8), turned to 90 degrees
- moved R1 87.6 mm to (163.2, 102.9), turned to -90 degrees
- moved R4 87.4 mm to (178.4, 102.9)
- moved D2 70.3 mm to (160.7, 62.9)
- moved R2 69.7 mm to (159.4, 102.9), turned to -90 degrees
- moved C2 68.7 mm to (174.7, 121.3)
- moved C1 67.3 mm to (167.6, 123.5), turned to 90 degrees
- moved D1 65.1 mm to (144.8, 62.9)
- moved R7 62.9 mm to (170.8, 110.5), turned to 90 degrees
- moved Q1 60.0 mm to (166.7, 116.8), turned to 90 degrees
- moved BAT1 17.7 mm to (139.7, 121.9), turned to 90 degrees
Routing:
- net Net-(D1-Pad2): track 0.00 -> 74.8 mm
- net Net-(D1-Pad1): track 0.00 -> 74.0 mm, vias 0 -> 1
- net VCC: track 0.00 -> 51.7 mm
- net Net-(D2-Pad2): track 0.00 -> 43.2 mm
- net Net-(C1-Pad1): track 0.00 -> 26.9 mm
- net Net-(C2-Pad1): track 0.00 -> 24.9 mm
- net Net-(R3-Pad1): track 0.00 -> 23.8 mm
- net Net-(R1-Pad2): track 0.00 -> 18.8 mm
- net Net-(BAT1-PadPos): track 0.00 -> 16.0 mm
- net Net-(Q1-Pad2): track 0.00 -> 13.0 mm
- net GND: track 0.00 -> 5.27 mm
- added copper zone on B.Cu, net GND
- added copper zone on F.Cu, net GND
Other:
- outline, holes or cut-outs redrawn
- board text added: "+"
- board text added: "ON"
